File: eagle/rPiMIDIShield/rPiMIDIShield.brd (EAGLE design)
At the start: 56 x 85 mm, 11 parts

Commit message: Added switches for 5v supply via MIDI
Parts:
- added LED1, LED2: (no value), led:LSU260
- added R1, R6: 4k7, resistor:0204/7
- added SV3: (no value), con-lstb:MA03-1
- moved SV2 80.5 mm to (6.35, 67.3)
Connections:
- new net N$1: LED2.A, MIDIIN.3, SV3.2
- new net N$13: LED2.K, R6.2
- new net N$5: LED1.K, R1.2
- net 5.0V: now also SV3.1
- net GND: now also MIDIIN.1, MIDIIN.2, MIDIOUT.1, R1.1, R6.1, SV3.3
- net N$2: now also LED1.A, MIDIOUT.3
Routing:
- net N$1: track 0.00 -> 36.0 mm
- net N$2: track 0.00 -> 17.8 mm
- net N$5: track 0.00 -> 8.82 mm
- net N$13: track 0.00 -> 8.27 mm
Changed lines of the file:
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@@
 <attribute name="VALUE" x="25.654" y="79.121" size="1.27" layer="27" ratio="10" rot="R180"/>
 </element>
-<element name="SV2" library="con-lstb" package="MA03-1" value="" x="4.572" y="-13.208">
-<attribute name="OC_NEWARK" value="unknown" x="4.572" y="-13.208" size="1.778" layer="27" display="off"/>
-<attribute name="MPN" value="" x="4.572" y="-13.208" size="1.778" layer="27" display="off"/>
-<attribute name="MF" value="" x="4.572" y="-13.208" size="1.778" layer="27" display="off"/>
-<attribute name="OC_FARNELL" value="unknown" x="4.572" y="-13.208" size="1.778" layer="27" display="off"/>
+<element name="SV2" library="con-lstb" package="MA03-1" value="" x="6.35" y="67.31">
+<attribute name="OC_NEWARK" value="unknown" x="6.35" y="67.31" size="1.778" layer="27" display="off"/>
+<attribute name="MPN" value="" x="6.35" y="67.31" size="1.778" layer="27" display="off"/>
+<attribute name="MF" value="" x="6.35" y="67.31" size="1.778" layer="27" display="off"/>
+<attribute name="OC_FARNELL" value="unknown" x="6.35" y="67.31" size="1.778" layer="27" display="off"/>
 </element>
+<element name="SV3" library="con-lstb" package="MA03-1" value="" x="6.35" y="12.954">
+<attribute name="OC_NEWARK" value="unknown" x="6.35" y="12.954" size="1.778" layer="27" display="off"/>
+<attribute name="MPN" value="" x="6.35" y="12.954" size="1.778" layer="27" display="off"/>
+<attribute name="MF" value="" x="6.35" y="12.954" size="1.778" layer="27" display="off"/>
+<attribute name="OC_FARNELL" value="unknown" x="6.35" y="12.954" size="1.778" layer="27" display="off"/>
+</element>
+<element name="LED1" library="led" package="LSU260" value="" x="3.81" y="73.152" rot="R90"/>
+<element name="R1" library="resistor" package="0204/7" value="4k7" x="8.89" y="75.692" rot="R90"/>
+<element name="LED2" library="led" package="LSU260" value="" x="3.556" y="7.112" rot="R270"/>
+<element name="R6" library="resistor" package="0204/7" value="4k7" x="9.144" y="5.08" rot="R270"/>
 </elements>
 <signals>
@@
 </polygon>
 <contactref element="SV2" pad="1"/>
-<wire x1="32.258" y1="56.134" x2="2.032" y2="-13.208" width="0" layer="19" extent="1-1"/>
+<contactref element="SV3" pad="1"/>
 </signal>
 <signal name="GND">
@@
 <contactref element="MIDIIN" pad="PE"/>
 <contactref element="SV2" pad="3"/>
-<wire x1="2.286" y1="27.686" x2="7.112" y2="-13.208" width="0" layer="19" extent="1-1"/>
+<contactref element="MIDIOUT" pad="1"/>
+<contactref element="MIDIIN" pad="1"/>
+<contactref element="MIDIIN" pad="2"/>
+<contactref element="SV3" pad="3"/>
+<contactref element="R1" pad="1"/>
+<contactref element="R6" pad="1"/>
 </signal>
 <signal name="SDA">
@@
 <signal name="N$2">
 <contactref element="SV2" pad="2"/>
+<contactref element="MIDIOUT" pad="3"/>
+<contactref element="LED1" pad="A"/>
+<wire x1="3.81" y1="71.882" x2="4.318" y2="71.882" width="0.4064" layer="16"/>
+<wire x1="4.318" y1="71.882" x2="6.35" y2="69.85" width="0.4064" layer="16"/>
+<wire x1="6.35" y1="69.85" x2="6.35" y2="67.31" width="0.4064" layer="16"/>
+<wire x1="6.35" y1="67.31" x2="6.35" y2="66.04" width="0.4064" layer="16"/>
+<wire x1="6.35" y1="66.04" x2="12.446" y2="59.944" width="0.4064" layer="16"/>
+<wire x1="12.446" y1="59.944" x2="12.446" y2="57.912" width="0.4064" layer="16"/>
+<wire x1="12.446" y1="57.912" x2="12.446" y2="58.166" width="0" layer="19" extent="16-16"/>
+</signal>
+<signal name="N$1">
+<contactref element="SV3" pad="2"/>
+<contactref element="MIDIIN" pad="3"/>
+<contactref element="LED2" pad="A"/>
+<wire x1="3.302" y1="8.382" x2="4.572" y2="8.382" width="0.4064" layer="1"/>
+<wire x1="4.572" y1="8.382" x2="6.35" y2="10.16" width="0.4064" layer="1"/>
+<wire x1="6.35" y1="10.16" x2="6.35" y2="18.542" width="0.4064" layer="1"/>
+<wire x1="6.35" y1="18.542" x2="4.826" y2="20.066" width="0.4064" layer="1"/>
+<wire x1="4.826" y1="20.066" x2="4.826" y2="27.94" width="0.4064" layer="1"/>
+<wire x1="4.826" y1="27.94" x2="12.446" y2="35.56" width="0.4064" layer="1"/>
+<wire x1="12.446" y1="35.56" x2="12.446" y2="38.608" width="0.4064" layer="1"/>
+<wire x1="12.446" y1="38.608" x2="12.446" y2="37.846" width="0" layer="19" extent="1-1"/>
+<wire x1="3.556" y1="8.382" x2="3.302" y2="8.382" width="0" layer="19" extent="1-1"/>
+<wire x1="6.35" y1="12.954" x2="6.35" y2="10.16" width="0" layer="19" extent="1-1"/>
+</signal>
+<signal name="N$5">
+<contactref element="LED1" pad="K"/>
+<contactref element="R1" pad="2"/>
+<wire x1="3.81" y1="74.422" x2="3.81" y2="77.216" width="0.4064" layer="16"/>
+<wire x1="3.81" y1="77.216" x2="6.096" y2="79.502" width="0.4064" layer="16"/>
+<wire x1="6.096" y1="79.502" x2="8.89" y2="79.502" width="0.4064" layer="16"/>
+</signal>
+<signal name="N$13">
+<wire x1="3.556" y1="5.588" x2="3.556" y2="4.064" width="0.4064" layer="1"/>
+<wire x1="3.556" y1="4.064" x2="6.35" y2="1.27" width="0.4064" layer="1"/>
+<contactref element="LED2" pad="K"/>
+<contactref element="R6" pad="2"/>
+<wire x1="6.35" y1="1.27" x2="9.144" y2="1.27" width="0.4064" layer="1"/>
+<wire x1="3.556" y1="5.588" x2="3.556" y2="5.842" width="0" layer="19" extent="1-1"/>
 </signal>
 </signals>
