File: eagle/channelSelectorDriver/channelSelctorDriver.sch (EAGLE design)
At the start: 10 parts, among them IC1 4025N, IC2 4071N, IC3 4071N

Commit message: Halved the size of the board. Much smaller, much cheaper.
Parts:
- added LED1: (no value), led:LEDLSU260
- added R1: (no value), resistor:R-US_0204/7
Connections:
- new net N$12: LED1.C, R1.2
- net GND: now also R1.1
- net VCC: now also LED1.A
Changed lines of the file:
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@@
 <part name="P+7" library="supply1" deviceset="VCC" device=""/>
 <part name="FRAME1" library="SparkFun" deviceset="FRAME-LETTER" device=""/>
+<part name="R1" library="resistor" deviceset="R-US_" device="0204/7"/>
+<part name="LED1" library="led" deviceset="LED" device="LSU260"/>
+<part name="P+8" library="supply1" deviceset="VCC" device=""/>
+<part name="GND5" library="supply1" deviceset="GND" device=""/>
 </parts>
 <sheets>
@@
 <instance part="FRAME1" gate="G$1" x="0" y="0"/>
 <instance part="FRAME1" gate="G$2" x="147.32" y="0"/>
+<instance part="R1" gate="G$1" x="172.72" y="63.5" rot="R90"/>
+<instance part="LED1" gate="G$1" x="172.72" y="76.2"/>
+<instance part="P+8" gate="VCC" x="172.72" y="86.36"/>
+<instance part="GND5" gate="1" x="172.72" y="50.8"/>
 </instances>
 <busses>
@@
 <wire x1="39.37" y1="142.24" x2="36.83" y2="142.24" width="0.1524" layer="91"/>
 </segment>
+<segment>
+<pinref part="LED1" gate="G$1" pin="A"/>
+<wire x1="172.72" y1="83.82" x2="172.72" y2="78.74" width="0.1524" layer="91"/>
+<pinref part="P+8" gate="VCC" pin="VCC"/>
+</segment>
 </net>
 <net name="GND" class="0">
@@
 <wire x1="129.54" y1="59.69" x2="134.62" y2="59.69" width="0.1524" layer="91"/>
 </segment>
-</net>
-<net name="N$22" class="0">
+<segment>
+<pinref part="R1" gate="G$1" pin="1"/>
+<wire x1="172.72" y1="58.42" x2="172.72" y2="53.34" width="0.1524" layer="91"/>
+<pinref part="GND5" gate="1" pin="GND"/>
+</segment>
+</net>
+<net name="N$10" class="0">
 <segment>
 <pinref part="KBD1_C" gate="G$1" pin="2"/>
@@
 </segment>
 </net>
-<net name="N$18" class="0">
+<net name="N$23" class="0">
 <segment>
 <pinref part="IC1" gate="A" pin="I2"/>
@@
 </segment>
 </net>
-<net name="N$17" class="0">
+<net name="N$24" class="0">
 <segment>
 <pinref part="KBD2_C" gate="G$1" pin="2"/>
@@
 </segment>
 </net>
-<net name="N$11" class="0">
+<net name="N$17" class="0">
 <segment>
 <pinref part="IC1" gate="B" pin="I1"/>
@@
 </segment>
 </net>
-<net name="N$12" class="0">
+<net name="N$4" class="0">
 <segment>
 <pinref part="KBD2_C" gate="G$1" pin="5"/>
@@
 </segment>
 </net>
-<net name="N$16" class="0">
+<net name="N$11" class="0">
 <segment>
 <pinref part="KBD3_C" gate="G$1" pin="2"/>
@@
 </segment>
 </net>
-<net name="N$4" class="0">
+<net name="N$18" class="0">
 <segment>
 <pinref part="IC1" gate="C" pin="I2"/>
@@
 </segment>
 </net>
+<net name="N$12" class="0">
+<segment>
+<pinref part="R1" gate="G$1" pin="2"/>
+<pinref part="LED1" gate="G$1" pin="C"/>
+<wire x1="172.72" y1="71.12" x2="172.72" y2="68.58" width="0.1524" layer="91"/>
+</segment>
+</net>
